File: dasbob.kicad_sch (KiCad schematic)
At the start: 68 parts, among them J1 TRRS LEFT, J2 TRRS LEFT, SW1 SW_Push, SW10 SW_Push, SW11 SW_Push, SW12 SW_Push, SW13 SW_Push, SW14 SW_Push, SW15 SW_Push, SW16 SW_Push, SW17 SW_Push, SW18 SW_Push, SW19 SW_Push, SW2 SW_Push, SW20 SW_Push, SW21 SW_Push, SW22 SW_Push, SW23 SW_Push, SW24 SW_Push, SW25 SW_Push, SW26 SW_Push, SW27 SW_Push, SW28 SW_Push, SW29 SW_Push, SW3 SW_Push, SW30 SW_Push, SW31 SW_Push, SW32 SW_Push, SW33 SW_Push, SW34 SW_Push, SW35 SW_Push, SW36 SW_Push, SW4 SW_Push, SW5 SW_Push, SW6 SW_Push, SW7 SW_Push, SW8 SW_Push, SW9 SW_Push, U1 Elite-C RIGHT, U2 Elite-C LEFT, U3 OLED1, U4 OLED2

Commit message: keybob v1
Parts:
- removed BZ1, BZ2: Buzzer, Buzzer_Beeper:Buzzer_Mallory_AST1109MLTRQ, symbol Device:Buzzer
- removed JP1: BLUETOOTH, keebio:JUMPER_SMD_2DUB, symbol Jumper:SolderJumper_2_Open
- removed JP2: WIRED, keebio:JUMPER_SMD_2DUB, symbol Jumper:SolderJumper_2_Open
- removed JP3: BLAUZAHN, keebio:JUMPER_SMD_2DUB, symbol Jumper:SolderJumper_2_Open
- removed JP4: KABEL, keebio:JUMPER_SMD_2DUB, symbol Jumper:SolderJumper_2_Open
- added BAT1_CONN1: Conn_01x02_Socket, symbol Connector:Conn_01x02_Socket
- BAT1: footprint Beibob:BAT -> thingymabob_library:Thingymabob_BAT
- J2: value TRRS LEFT -> TRRS RIGHT
- RST1: value RESET BUTTON RIGHT -> RESET BUTTON LEFT
- TAB1: footprint Beibob:BAT -> thingymabob_library:Thingymabob_TAB
- TSR1: value RESET BUTTON LEFT -> RESET BUTTON RIGHT
- U1: value Elite-C RIGHT -> Elite-C LEFT
- U2: value Elite-C LEFT -> Elite-C RIGHT
Connections:
- net C6 is gone; now on net 7: U1.8 (5/PC6)
- net C6a is gone; now on net 9a: U2.8 (5/PC6)
- net C7 is gone; now on net 12: U1.27 (C7)
- net C7a is gone; now on net 16a: U2.27 (C7)
- net 1: now also U1.18 (A1/PF6); no longer U1.26 (D5)
- net 10: no longer U1.18 (A1/PF6)
- net 10a: now also U2.17 (A0/PF7); no longer U2.18 (A1/PF6)
- net 11: now also U1.26 (D5)
- net 11a: now also U2.26 (D5); no longer U2.13 (10/PB6)
- net 12a: now also U2.25 (B7); no longer U2.14 (16/PB2)
- net 13a: now also U2.12 (9/PB5); no longer U2.10 (7/PE6)
- net 14a: now also U2.11 (8/PB4); no longer U2.15 (14/PB3)
- net 15a: now also U2.10 (7/PE6); no longer U2.9 (6/PD7)
- net 16: now also U1.25 (B7); no longer U1.29 (F0)
- net 16a: no longer U2.29 (F0)
- net 17a: now also U2.14 (16/PB2); no longer U2.12 (9/PB5)
- net 18a: now also U2.13 (10/PB6); no longer U2.11 (8/PB4)
- net 1a: now also U2.7 (4/PD4); no longer U2.26 (D5)
- net 2a: now also U2.18 (A1/PF6); no longer U2.19 (A2/PF5)
- net 3: now also U1.7 (4/PD4); no longer U1.25 (B7)
- net 3a: now also U2.19 (A2/PF5); no longer U2.25 (B7)
- net 6a: now also U2.15 (14/PB3); no longer U2.16 (15/PB1)
- net 7a: now also U2.9 (6/PD7)
- net 8a: now also U2.16 (15/PB1); no longer U2.17 (A0/PF7)
- net 9: no longer U1.7 (4/PD4)
- net 9a: no longer U2.7 (4/PD4)
- net BAT: now also BAT1_CONN1.1 (Pin_1)
- net GND: now also BAT1_CONN1.2 (Pin_2)
